File: sprayGun_PCB/sprayGun_PCB.kicad_sch (KiCad schematic)
At the start: 31 parts

Commit message: Rev A done
Parts:
- added C5: 10uF, symbol Device:C_Small
- added C6, C7, C8: (no value), symbol Device:C_Small
- added J15: ESC terminal, TerminalBlock_Phoenix:TerminalBlock_Phoenix_MKDS-3-3-5.08_1x03_P5.08mm_Horizontal, symbol Connector_Generic:Conn_01x03
- added J16: VESC terminal, TerminalBlock_Phoenix:TerminalBlock_Phoenix_MKDS-3-3-5.08_1x03_P5.08mm_Horizontal, symbol Connector_Generic:Conn_01x03
- added J17: SERVO terminal, TerminalBlock_Phoenix:TerminalBlock_Phoenix_MKDS-3-3-5.08_1x03_P5.08mm_Horizontal, symbol Connector_Generic:Conn_01x03
- added J18: (no value), symbol Connector_Generic:Conn_01x06
- added J19: (no value), TerminalBlock_Phoenix:TerminalBlock_Phoenix_MKDS-3-2-5.08_1x02_P5.08mm_Horizontal, symbol Connector_Generic:Conn_01x02
- C1: renamed from C?; value (none) -> 33uF; footprint (none) -> Capacitor_THT:CP_Radial_D6.3mm_P2.50mm
- C2: renamed from C?; value (none) -> 0.1uF; footprint (none) -> Capacitor_THT:CP_Radial_D5.0mm_P2.50mm
- C3, C4: renamed from C?; footprint (none) -> Capacitor_THT:CP_Radial_Tantal_D5.0mm_P2.50mm
- D1, D2, D3: renamed from D?; footprint (none) -> LED_THT:LED_D5.0mm
- IC1: renamed from IC?; value (none) -> L78S05CV; footprint (none) -> libraries:L78S05CV
- J1: renamed from J?; value (none) -> PWR IN; footprint (none) -> TerminalBlock_Phoenix:TerminalBlock_Phoenix_MKDS-3-2-5.08_1x02_P5.08mm_Horizontal
- J10: renamed from J?; value (none) -> Analog IO; footprint (none) -> TerminalBlock_Phoenix:TerminalBlock_Phoenix_MKDS-3-8-5.08_1x08_P5.08mm_Horizontal
- J11: renamed from J?; value (none) -> Digital IO; footprint (none) -> TerminalBlock_Phoenix:TerminalBlock_Phoenix_MKDS-3-10-5.08_1x10_P5.08mm_Horizontal
- J12, J14: renamed from J?; footprint (none) -> Connector_PinHeader_2.54mm:PinHeader_1x02_P2.54mm_Vertical
- J13: renamed from J?; footprint (none) -> TerminalBlock_Phoenix:TerminalBlock_Phoenix_MKDS-3-2-5.08_1x02_P5.08mm_Horizontal
- J2: renamed from J?; footprint (none) -> Connector_PinSocket_2.54mm:PinSocket_1x10_P2.54mm_Vertical
- J3: renamed from J?; value VL53L0X -> (none)
- J4: renamed from J?; value (none) -> 5V rail; footprint (none) -> TerminalBlock_Phoenix:TerminalBlock_Phoenix_MKDS-3-4-5.08_1x04_P5.08mm_Horizontal
- J5: renamed from J?; value (none) -> GND rail; footprint (none) -> TerminalBlock_Phoenix:TerminalBlock_Phoenix_MKDS-3-4-5.08_1x04_P5.08mm_Horizontal
- J6: renamed from J?; value ESC -> ESC header; footprint (none) -> Connector_PinHeader_2.54mm:PinHeader_1x03_P2.54mm_Vertical
- J7: renamed from J?; value VESC -> VESC header; footprint (none) -> Connector_PinHeader_2.54mm:PinHeader_1x03_P2.54mm_Vertical
- J8: renamed from J?; value Servo -> SERVO header; footprint (none) -> Connector_PinHeader_2.54mm:PinHeader_1x03_P2.54mm_Vertical
- J9: renamed from J?; value (none) -> 15V rail; footprint (none) -> TerminalBlock_Phoenix:TerminalBlock_Phoenix_MKDS-3-4-5.08_1x04_P5.08mm_Horizontal
- R1, R2, R4, R5: renamed from R?; footprint (none) -> Resistor_THT:R_Axial_DIN0207_L6.3mm_D2.5mm_P10.16mm_Horizontal
- R3: renamed from R?; value (none) -> 1k; footprint (none) -> Resistor_THT:R_Axial_DIN0207_L6.3mm_D2.5mm_P10.16mm_Horizontal
- U2: renamed from U?; footprint SOIC127P599X175-8N -> libraries:SN65HVD266D
- Y1: renamed from Y?; footprint (none) -> Crystal:Crystal_HC49-4H_Vertical
- gave numbers to parts that had none: 2
Connections:
- net +15V: now also J19.1 (Pin_1); no longer J1.1 (Pin_1)
- net +5VA: now also C5.1, C6.1, C7.1, C8.1, J17.2 (Pin_2), J18.1 (Pin_1)
- net ESC: now also J15.1 (Pin_1)
- net GND: now also C5.2, C6.2, C7.2, C8.2, J15.3 (Pin_3), J16.3 (Pin_3), J17.3 (Pin_3), J18.2 (Pin_2)
- net SCL: now also J18.3 (Pin_3)
- net SDA: now also J18.4 (Pin_4)
- net SERVO: now also J17.1 (Pin_1)
- net VESC: now also J16.1 (Pin_1)
- net TXD: now reaches U1.1 (TXCAN), U2.1 (TXD)
- net RXD: now reaches U1.2 (RXCAN), U2.4 (RXD)
- net OSC2: now reaches C3.2, U1.7 (OSC2), Y1.1
- net OSC1: now reaches C4.2, U1.8 (OSC1), Y1.2
- net CANL: now reaches J13.1 (Pin_1), J14.1 (Pin_1), R4.2, U2.6 (CANL)
- net CANH: now reaches J12.2 (Pin_2), J13.2 (Pin_2), J14.2 (Pin_2), U2.7 (CANH)
- new net: J1.1 (Pin_1), J19.2 (Pin_2)
- no-connect marks 18 -> 25
Other:
- note added: "ESC header"
- note added: "ESC terminal"
- note added: "Output Connectors and IO Breakouts"
- note added: "SERVO header"
- note added: "SERVO terminal"
- note added: "VESC header"
- note added: "VESC terminal"
- note removed: "ESC"
- note removed: "Output Connectors"
- note removed: "SERVO"
- note removed: "VESC"
- moved on the sheet: C1, C2, C3, C4, D3, IC1, J10, J11, J12, J13, J14, J3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

Commit message: This revision was sent to JLC for production.
Parts:
- removed U2: SN65HVD266D, libraries:SN65HVD266D, symbol SN65HVD266D:SN65HVD266D
- added U2: (no value), symbol SN65HVD253D:SN65HVD253D
Connections:
- net +5V: now also J17.2 (Pin_2), J8.2 (Pin_2)
- net +5VA: now also U2.3 (VCC); no longer J17.2 (Pin_2), J8.2 (Pin_2)
- net CANH: now also U2.7 (CANH)
- net CANL: now also U2.6 (CANL)
- net GND: now also U2.2 (GND), U2.5 (AB), U2.8 (S)
- net RXD: now also U2.4 (RXD)
- net TXD: now also U2.1 (TXD)
- no-connect marks 25 -> 24
Other:
- note removed: "S (pin 8) set to LOW = Normal Mode"
- moved on the sheet: C7, C8, J12, J13, J14, R4

Commit message: Exported step file o of PCB.
Parts:
- C5: footprint (none) -> Capacitor_THT:CP_Radial_D5.0mm_P2.00mm
- C6, C8: value (none) -> 0.1uF; footprint (none) -> Capacitor_THT:CP_Radial_D5.0mm_P2.50mm
- C7: value (none) -> 10uF; footprint (none) -> Capacitor_THT:CP_Radial_D5.0mm_P2.00mm
- D1: value (none) -> LED1
- D2: value (none) -> LED2
- D3: value (none) -> PWR LED
- J18: value (none) -> VL53L0X 2; footprint (none) -> Connector_JST:JST_XH_B6B-XH-A_1x06_P2.50mm_Vertical
- J19: value (none) -> E-stop
- J3: value (none) -> VL53L0X 1; footprint (none) -> Connector_JST:JST_XH_B6B-XH-A_1x06_P2.50mm_Vertical
- U2: value (none) -> SN65HVD253D; footprint (none) -> libraries:SN65HVD253D
Other:
- added sheet CAN bus interface (untitled.kicad_sch)
- added sheet Power Regulation (power_regulation.kicad_sch)
